File: LowNoiseDual5W/LowNoiseDual5W.kicad_pcb (KiCad board)
At the start: 2 copper layers, 116 x 45 mm, 63 parts, among them J1 B3B-XH-A, J10 Screw_Terminal_01x02, J11 B2B-XH-A, J12 B2B-XH-A, J13 B2B-XH-A, J2 B3B-XH-A, J3 B3B-XH-A, J5 B2B-XH-A, J6 Screw_Terminal_01x02, J7 Screw_Terminal_01x02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

Commit message: Add fiducials
Parts:
- added FID1: Fiducial, Fiducial:Fiducial_0.5mm_Mask1mm, F.Cu at (69.0, 39.2)
- added FID2: Fiducial, Fiducial:Fiducial_0.5mm_Mask1mm, F.Cu at (162.2, 74.5)
- added FID3: Fiducial, Fiducial:Fiducial_0.5mm_Mask1mm, F.Cu at (76.8, 74.2)
Changed lines of the file:
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@@
   )
   (paper "A4")
+  (title_block
+    (comment 4 "AISLER Project ID: TQEIXWXZ")
+  )
   (layers
     (0 "F.Cu" signal)
@@
     (fp_line (start 4.95 3.4) (end 4.95 -2.35)
       (stroke (width 0.1) (type solid)) (layer "F.Fab"))
-    (pad "1" thru_hole roundrect (at 0 0 270) (size 1.7 2) (drill 1) (layers "*.Cu" "*.Mask") (roundrect_rratio 0.147059)
+    (pad "1" thru_hole roundrect (at 0 0 270) (size 1.7 2) (drill 1) (layers "*.Cu" "*.Mask") (roundrect_rratio 0.1470588235)
       (net 9 "Net-(D3-A)") (pinfunction "Pin_1") (pintype "passive"))
     (pad "2" thru_hole oval (at 2.5 0 270) (size 1.7 2) (drill 1) (layers "*.Cu" "*.Mask")
@@
     )
   )
+  (footprint "Fiducial:Fiducial_0.5mm_Mask1mm" (layer "F.Cu")
+    (at 69 39.25)
+    (descr "Circular Fiducial, 0.5mm bare copper, 1mm soldermask opening (Level C)")
+    (tags "fiducial")
+    (property "Sheetfile" "LowNoiseDual5W.kicad_sch")
+    (property "Sheetname" "")
+    (property "ki_description" "Fiducial Marker")
+    (property "ki_keywords" "fiducial marker")
+    (attr smd)
+    (fp_text reference "FID1" (at 0 -1.5) (layer "F.SilkS")
+        (effects (font (size 1 1) (thickness 0.15)))
+    )
+    (fp_text value "Fiducial" (at 0 1.5) (layer "F.Fab")
+        (effects (font (size 1 1) (thickness 0.15)))
+    )
+    (fp_text user "${REFERENCE}" (at 0 0) (layer "F.Fab")
+        (effects (font (size 0.2 0.2) (thickness 0.04)))
+    )
+    (fp_circle (center 0 0) (end 0.75 0)
+      (stroke (width 0.05) (type solid)) (fill none) (layer "F.CrtYd"))
+    (fp_circle (center 0 0) (end 0.5 0)
+      (stroke (width 0.1) (type solid)) (fill none) (layer "F.Fab"))
+    (pad "" smd circle (at 0 0) (size 0.5 0.5) (layers "F.Cu" "F.Mask")
+      (solder_mask_margin 0.25) (clearance 0.25))
+  )
   (footprint "Resistor_SMD:R_0603_1608Metric" (layer "F.Cu")
     (at 141.7 64.8)
@@
     )
   )
+  (footprint "Fiducial:Fiducial_0.5mm_Mask1mm" (layer "F.Cu")
+    (at 162.25 74.5)
+    (descr "Circular Fiducial, 0.5mm bare copper, 1mm soldermask opening (Level C)")
+    (tags "fiducial")
+    (property "Sheetfile" "LowNoiseDual5W.kicad_sch")
+    (property "Sheetname" "")
+    (property "ki_description" "Fiducial Marker")
+    (property "ki_keywords" "fiducial marker")
+    (attr smd)
+    (fp_text reference "FID2" (at 0 -1.5) (layer "F.SilkS")
+        (effects (font (size 1 1) (thickness 0.15)))
+    )
+    (fp_text value "Fiducial" (at 0 1.5) (layer "F.Fab")
+        (effects (font (size 1 1) (thickness 0.15)))
+    )
+    (fp_text user "${REFERENCE}" (at 0 0) (layer "F.Fab")
+        (effects (font (size 0.2 0.2) (thickness 0.04)))
+    )
+    (fp_circle (center 0 0) (end 0.75 0)
+      (stroke (width 0.05) (type solid)) (fill none) (layer "F.CrtYd"))
+    (fp_circle (center 0 0) (end 0.5 0)
+      (stroke (width 0.1) (type solid)) (fill none) (layer "F.Fab"))
+    (pad "" smd circle (at 0 0) (size 0.5 0.5) (layers "F.Cu" "F.Mask")
+      (solder_mask_margin 0.25) (clearance 0.25))
+  )
   (footprint "Resistor_SMD:R_0603_1608Metric" (layer "F.Cu")
     (at 91.6375 64.0625)
@@
     (fp_line (start 2.5 2.5) (end -2.5 2.5)
       (stroke (width 0.1) (type solid)) (layer "F.Fab"))
-    (pad "" smd roundrect (at -0.79 -0.79) (size 1.27 1.27) (layers "F.Paste") (roundrect_rratio 0.19685))
-    (pad "" smd roundrect (at -0.79 0.79) (size 1.27 1.27) (layers "F.Paste") (roundrect_rratio 0.19685))
-    (pad "" smd roundrect (at 0.79 -0.79) (size 1.27 1.27) (layers "F.Paste") (roundrect_rratio 0.19685))
-    (pad "" smd roundrect (at 0.79 0.79) (size 1.27 1.27) (layers "F.Paste") (roundrect_rratio 0.19685))
+    (pad "" smd roundrect (at -0.79 -0.79) (size 1.27 1.27) (layers "F.Paste") (roundrect_rratio 0.1968503937))
+    (pad "" smd roundrect (at -0.79 0.79) (size 1.27 1.27) (layers "F.Paste") (roundrect_rratio 0.1968503937))
+    (pad "" smd roundrect (at 0.79 -0.79) (size 1.27 1.27) (layers "F.Paste") (roundrect_rratio 0.1968503937))
+    (pad "" smd roundrect (at 0.79 0.79) (size 1.27 1.27) (layers "F.Paste") (roundrect_rratio 0.1968503937))
     (pad "1" smd roundrect (at -2.3625 -1.3) (size 1.025 0.35) (layers "F.Cu" "F.Paste" "F.Mask") (roundrect_rratio 0.25)
       (net 1 "+5V") (pinfunction "OUT") (pintype "power_out"))
@@
     (fp_line (start 3.95 2.8) (end 3.95 -1.7)
       (stroke (width 0.1) (type solid)) (layer "F.Fab"))
-    (pad "1" thru_hole roundrect (at 0 0 90) (size 1.2 1.75) (drill 0.75) (layers "*.Cu" "*.Mask") (roundrect_rratio 0.208333)
+    (pad "1" thru_hole roundrect (at 0 0 90) (size 1.2 1.75) (drill 0.75) (layers "*.Cu" "*.Mask") (roundrect_rratio 0.2083333333)
       (net 29 "Net-(J12-Pin_1)") (pinfunction "Pin_1") (pintype "passive"))
     (pad "2" thru_hole oval (at 2 0 90) (size 1.2 1.75) (drill 0.75) (layers "*.Cu" "*.Mask")
@@
     (fp_line (start 2.5 2.5) (end -2.5 2.5)
       (stroke (width 0.1) (type solid)) (layer "F.Fab"))
-    (pad "" smd roundrect (at -0.79 -0.79) (size 1.27 1.27) (layers "F.Paste") (roundrect_rratio 0.19685))
-    (pad "" smd roundrect (at -0.79 0.79) (size 1.27 1.27) (layers "F.Paste") (roundrect_rratio 0.19685))
-    (pad "" smd roundrect (at 0.79 -0.79) (size 1.27 1.27) (layers "F.Paste") (roundrect_rratio 0.19685))
-    (pad "" smd roundrect (at 0.79 0.79) (size 1.27 1.27) (layers "F.Paste") (roundrect_rratio 0.19685))
+    (pad "" smd roundrect (at -0.79 -0.79) (size 1.27 1.27) (layers "F.Paste") (roundrect_rratio 0.1968503937))
+    (pad "" smd roundrect (at -0.79 0.79) (size 1.27 1.27) (layers "F.Paste") (roundrect_rratio 0.1968503937))
+    (pad "" smd roundrect (at 0.79 -0.79) (size 1.27 1.27) (layers "F.Paste") (roundrect_rratio 0.1968503937))
+    (pad "" smd roundrect (at 0.79 0.79) (size 1.27 1.27) (layers "F.Paste") (roundrect_rratio 0.1968503937))
     (pad "1" smd roundrect (at -2.3625 -1.3) (size 1.025 0.35) (layers "F.Cu" "F.Paste" "F.Mask") (roundrect_rratio 0.25)
       (net 5 "-5V") (pinfunction "OUT") (pintype "power_out"))
@@
     )
   )
+  (footprint "Fiducial:Fiducial_0.5mm_Mask1mm" (layer "F.Cu")
+    (at 76.75 74.25)
+    (descr "Circular Fiducial, 0.5mm bare copper, 1mm soldermask opening (Level C)")
+    (tags "fiducial")
+    (property "Sheetfile" "LowNoiseDual5W.kicad_sch")
+    (property "Sheetname" "")
+    (property "ki_description" "Fiducial Marker")
+    (property "ki_keywords" "fiducial marker")
+    (attr smd)
+    (fp_text reference "FID3" (at 0 -1.5) (layer "F.SilkS")
+        (effects (font (size 1 1) (thickness 0.15)))
+    )
+    (fp_text value "Fiducial" (at 0 1.5) (layer "F.Fab")
+        (effects (font (size 1 1) (thickness 0.15)))
+    )
+    (fp_text user "${REFERENCE}" (at 0 0) (layer "F.Fab")
+        (effects (font (size 0.2 0.2) (thickness 0.04)))
+    )
+    (fp_circle (center 0 0) (end 0.75 0)
+      (stroke (width 0.05) (type solid)) (fill none) (layer "F.CrtYd"))
+    (fp_circle (center 0 0) (end 0.5 0)
+      (stroke (width 0.1) (type solid)) (fill none) (layer "F.Fab"))
+    (pad "" smd circle (at 0 0) (size 0.5 0.5) (layers "F.Cu" "F.Mask")
+      (solder_mask_margin 0.25) (clearance 0.25))
+  )
   (footprint "MountingHole:MountingHole_3.2mm_M3_ISO7380" (layer "F.Cu")
