File: LowNoiseDual5W/LowNoiseDual5W.kicad_sch (KiCad schematic)
At the start: 0 parts

Commit message: Implement low noise dual 5W power supply
Parts:
- added C1, C12, C9: 1uF, Resistor_SMD:R_0603_1608Metric, symbol Device:C_Small
- added C10, C11, C14, C15, C16, C17, C19, C20, C21, C22, C3, C4, C5, C6, C7, C8: 22uF 16V, Capacitor_SMD:C_1206_3216Metric, symbol Device:C_Small
- added C13: 1nF, Resistor_SMD:R_0603_1608Metric, symbol Device:C_Small
- added C18: 100nF, Resistor_SMD:R_0603_1608Metric, symbol Device:C_Small
- added C2: 10uF, Resistor_SMD:R_0603_1608Metric, symbol Device:C_Small
- added C23: 10pF, Resistor_SMD:R_0603_1608Metric, symbol Device:C_Small
- added D1, D2: SMAJ5.0A, Diode_SMD:D_SMA, symbol Diode:SMAJ5.0A
- added D3: SS210, Diode_SMD:D_SMA, symbol Uli-Diode:SS210
- added D4: SMAJ12A, Diode_SMD:D_SMA, symbol Uli-Diode:SMAJ12A
- added D5, D6: SMAJ12.0A, Diode_SMD:D_SMA, symbol Diode:SMAJ5.0A
- added FB1, FB2, FB3, FB4: 742792097, Inductor_SMD:L_0805_2012Metric, symbol Device:FerriteBead_Small
- added H1, H2, H3, H4: MountingHole, MountingHole:MountingHole_3.2mm_M3_ISO7380, symbol Mechanical:MountingHole
- added J1, J2, J3, J9: B3B-XH-A, Connector_JST:JST_XH_B3B-XH-A_1x03_P2.50mm_Vertical, symbol Connector:Conn_01x03_Pin
- added J10, J6, J7, J8: Screw_Terminal_01x02, TerminalBlock_Phoenix:TerminalBlock_Phoenix_MKDS-1,5-2-5.08_1x02_P5.08mm_Horizontal, symbol Connector:Screw_Terminal_01x02
- added J11, J13, J5: B2B-XH-A, Connector_JST:JST_XH_B2B-XH-A_1x02_P2.50mm_Vertical, symbol Connector:Conn_01x02_Pin
- added J12: B2B-XH-A, Connector_JST:JST_PH_B2B-PH-K_1x02_P2.00mm_Vertical, symbol Connector:Conn_01x02_Pin
- added J4: Jack-DC, Connector_BarrelJack:BarrelJack_GCT_DCJ200-10-A_Horizontal, symbol Connector:Jack-DC
- added L1: L_Small, Uli-RAM:L_SXN_SMDRI127, symbol Device:L_Small
- added R1: 10k, Resistor_SMD:R_0603_1608Metric, symbol Device:R_Small
- added R2: 25.5k, Resistor_SMD:R_0603_1608Metric, symbol Device:R_Small
- added R3: 100k, Resistor_SMD:R_0603_1608Metric, symbol Device:R_Small
- added R4, R6: 332k, Resistor_SMD:R_0603_1608Metric, symbol Device:R_Small
- added R5, R7: 102k, Resistor_SMD:R_0603_1608Metric, symbol Device:R_Small
- added SW1: RST, Button_Switch_SMD:SW_SPST_TL3342, symbol Switch:SW_Push
- added SW2: SW_SPDT, Button_Switch_SMD:SW_DPDT_CK_JS202011JCQN, symbol Switch:SW_SPDT
- added U1: TPS7A4701xRGW, Package_DFN_QFN:Texas_S-PVQFN-N20_EP3.15x3.15mm, symbol Uli-LinReg:TPS7A4701xRGW
- added U2: TPS7A3301RGW, Package_DFN_QFN:Texas_S-PVQFN-N20_EP3.15x3.15mm, symbol Uli-LinReg:TPS7A3301RGW
- added U3: TPS62932, Package_TO_SOT_SMD:SOT-583-8, symbol Uli-RegSw:TPS62932
- added U4: NSD10-xxDyy, Uli-DCDC:Converter_DCDC_MeanWell_NSD10_THT, symbol Uli-DCDC:NSD10-xxDyy
Connections:
- new net: C7.2, C8.1, FB1.2, U1.13 (EN), U1.15 (IN), U1.16 (IN)
- new net: C1.1, U1.14 (NR)
- new net: C2.2, R1.1, R2.2, U1.3 (SENSE/FB)
- new net: J12.1 (Pin_1), SW1.1, SW2.3 (C), U4.6 (Control)
- new net: C12.1, U2.14 (NR/SS)
- new net: C13.2, R4.2, R5.1, U2.3 (FB)
- new net: R3.1, U3.1 (RT)
- new net: C23.2, R6.2, R7.1, U3.8 (FB)
- new net: D3.2 (A), J13.1 (Pin_1), J4.1, J5.1 (Pin_1), J8.1 (Pin_1)
- new net: C9.1, U3.7 (SS)
- new net: C18.1, U3.6 (BST)
- new net: C18.2, L1.1, U3.5 (SW)
- new net: C19.2, C20.1, FB3.2, U3.2 (EN), U3.3 (VIN)
- new net: C22.1, FB4.1, L1.2
- new net +12V: D5.1 (A1), FB1.1, FB3.1, J9.1 (Pin_1), U4.3 (+OUT)
- new net +5V: C2.1, C3.1, C4.2, C5.2, C6.1, D1.1 (A1), J1.1 (Pin_1), J2.1 (Pin_1), J3.1 (Pin_1), J6.1 (Pin_1), R2.1, U1.1 (OUT), U1.20 (OUT)
- new net +5VD: C21.1, C23.1, FB4.2, J10.1 (Pin_1), J11.1 (Pin_1), R6.1
- new net -12V: D6.2 (A2), FB2.1, J9.3 (Pin_3), U4.5 (-OUT)
- new net -5V: C13.1, C14.2, C15.1, C16.2, C17.1, D2.2 (A2), J1.3 (Pin_3), J2.3 (Pin_3), J3.3 (Pin_3), J7.2 (Pin_2), R4.1, U2.1 (OUT), U2.20 (OUT)
- new net 12V_{In}: D3.1 (K), D4.1 (A1), U4.1 (+IN)
- new net GND: C1.2, C10.1, C11.2, C12.2, C14.1, C15.2, C16.1, C17.2, C19.1, C20.2, C21.2, C22.2, C3.2, C4.1, C5.1, C6.2, C7.1, C8.2, C9.2, D1.2 (A2), D2.1 (A1), D5.2 (A2), D6.1 (A1), J1.2 (Pin_2), J10.2 (Pin_2), J11.2 (Pin_2), J2.2 (Pin_2), J3.2 (Pin_2), J6.2 (Pin_2), J7.1 (Pin_1), J9.2 (Pin_2), R1.2, R3.2, R5.2, R7.2, U1.21 (EP), U1.7 (GND), U2.21 (EP), U2.7 (GND), U3.4 (GND), U4.4 (Common)
- new net GNDPWR: D4.2 (A2), J12.2 (Pin_2), J13.2 (Pin_2), J5.2 (Pin_2), J8.2 (Pin_2), SW1.2, SW2.2 (B), U4.2 (-IN)
- new net IN: C10.2, C11.1, FB2.2, U2.13 (EN), U2.15 (IN), U2.16 (IN)
- no-connect marks 0 -> 9
Other:
- note added: "+5V@1A low noise analog supply"
- note added: "-5V@-1A low noise analog supply"
- note added: "1nF Cff provides low PSRR in 100kHz..1MHz range which suppresses input DC/DC noise"
- note added: "5V@2A digital auxiliary supply"
- note added: "Closed = off"
- note added: "Daisy-chain power"
- note added: "Datasheet suggestion resistors for +5V. ANY-OUT not used to allow easier change of voltages"
- note added: "Datasheet suggestion resistors for -5V"
- note added: "Ferrite selection: 1A current Maximum impedance @1MHz"
- note added: "Main isolating DC/DC"
- note added: "Momentary reset"
- note added: "OVP 12V"
- note added: "OVP 5V"
- note added: "Output connectors"
- note added: "f_{SW} = 250kHz for best PSRR by LDOs"
- note added: "~100uF Cout for maximum PSRR"

Commit message: Add fiducials
Parts:
- added FID1, FID2, FID3: Fiducial, Fiducial:Fiducial_0.5mm_Mask1mm, symbol Mechanical:Fiducial
Changed lines of the file:
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@@
+    )
+  )
+  (symbol (lib_id "Mechanical:Fiducial") (at 97.155 19.05 0) (unit 1)
+    (in_bom yes) (on_board yes) (dnp no) (fields_autoplaced)
+    (property "Reference" "FID2" (at 99.695 17.78 0)
+      (effects (font (size 1.27 1.27)) (justify left))
+    )
+    (property "Value" "Fiducial" (at 99.695 20.32 0)
+      (effects (font (size 1.27 1.27)) (justify left))
+    )
+    (property "Footprint" "Fiducial:Fiducial_0.5mm_Mask1mm" (at 97.155 19.05 0)
+      (effects (font (size 1.27 1.27)) hide)
+    )
+    (property "Datasheet" "~" (at 97.155 19.05 0)
+      (effects (font (size 1.27 1.27)) hide)
+    )
+    (instances
+      (project "LowNoiseDual5W"
+        (path "/df87b081-37a2-452c-8581-7eff2c408a17"
+          (reference "FID2") (unit 1)
+        )
+      )
     )
   )
@@
         (path "/df87b081-37a2-452c-8581-7eff2c408a17"
           (reference "#PWR065") (unit 1)
+        )
+      )
+    )
+  )
+  (symbol (lib_id "Mechanical:Fiducial") (at 78.74 19.05 0) (unit 1)
+    (in_bom yes) (on_board yes) (dnp no) (fields_autoplaced)
+    (property "Reference" "FID1" (at 81.28 17.78 0)
+      (effects (font (size 1.27 1.27)) (justify left))
+    )
+    (property "Value" "Fiducial" (at 81.28 20.32 0)
+      (effects (font (size 1.27 1.27)) (justify left))
+    )
+    (property "Footprint" "Fiducial:Fiducial_0.5mm_Mask1mm" (at 78.74 19.05 0)
+      (effects (font (size 1.27 1.27)) hide)
+    )
+    (property "Datasheet" "~" (at 78.74 19.05 0)
+      (effects (font (size 1.27 1.27)) hide)
+    )
+    (instances
+      (project "LowNoiseDual5W"
+        (path "/df87b081-37a2-452c-8581-7eff2c408a17"
+          (reference "FID1") (unit 1)
         )
       )
@@
         )
       )
+    )
+  )
+  (symbol (lib_id "Mechanical:Fiducial") (at 118.11 19.05 0) (unit 1)
+    (in_bom yes) (on_board yes) (dnp no) (fields_autoplaced)
+    (property "Reference" "FID3" (at 120.65 17.78 0)
+      (effects (font (size 1.27 1.27)) (justify left))
+    )
+    (property "Value" "Fiducial" (at 120.65 20.32 0)
+      (effects (font (size 1.27 1.27)) (justify left))
+    )
+    (property "Footprint" "Fiducial:Fiducial_0.5mm_Mask1mm" (at 118.11 19.05 0)
+      (effects (font (size 1.27 1.27)) hide)
+    )
+    (property "Datasheet" "~" (at 118.11 19.05 0)
+      (effects (font (size 1.27 1.27)) hide)
+    )
+    (instances
+      (project "LowNoiseDual5W"
+        (path "/df87b081-37a2-452c-8581-7eff2c408a17"
+          (reference "FID3") (unit 1)
+        )
+      )
